File: hardware/MUSE-PEDAL.kicad_sch (KiCad schematic)
At the start: 45 parts, among them Q1 BC547C, Q2 BC547C, Q3 BC547C, Q4 BC547C

Commit message: f
Parts:
- removed C14: 100nF, symbol Device:C
- added C15: 100nF, symbol Device:C
Connections:
- net at C13.2, D4.1 (K), D5.2 (A)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: now also C15.1
- net at R22.2: now also C15.2
Other:
- moved on the sheet: R14, R20, R22
